File: hardware/eagle-project/beaglebone_rotor_control_cape.sch (EAGLE design)
At the start: 59 parts, among them IC1 TLC2264CDU, IC2 MCP4901, IC3 MAX3232ESE, IC4 TLC2264CDU, IC5 MCP4901, IC6 TLC2264CDU, Q1 SQ2348ES-T1-GE3, Q2 SQ2348ES-T1-GE3, Q3 SQ2348ES-T1-GE3, Q4 SQ2348ES-T1-GE3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

Commit message: Added USB connector
Parts:
- added X5: USBDEV, con-usbbuchse:USBDEV
Connections:
- net GND: now also X5.GND
Other:
- note added: "Rotor controller supply control"
- note added: "USB-Buchse für Master-Slave Steckdosenleiste"
Changed lines of the file:
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@@
 <part name="X4" library="con-te-dsub" deviceset="DSUB9" device=""/>
 <part name="GND31" library="supply1" deviceset="GND" device=""/>
+<part name="FRAME5" library="frames_2" deviceset="A4L-LOC" device=""/>
+<part name="X5" library="con-usbbuchse" deviceset="USBDEV" device=""/>
+<part name="GND32" library="supply1" deviceset="GND" device=""/>
+<part name="P+7" library="supply1" deviceset="+5V" device=""/>
 </parts>
 <sheets>
@@
 </segment>
 </net>
+</nets>
+</sheet>
+<sheet>
+<plain>
+<text x="179.07" y="20.32" size="2.54" layer="94">Rotor controller supply control</text>
+<text x="30.48" y="139.7" size="2.54" layer="95">USB-Buchse für Master-Slave Steckdosenleiste</text>
+</plain>
+<instances>
+<instance part="FRAME5" gate="G$1" x="0" y="0"/>
+<instance part="X5" gate="G$1" x="83.82" y="101.6"/>
+<instance part="GND32" gate="1" x="71.12" y="88.9"/>
+<instance part="P+7" gate="1" x="71.12" y="116.84"/>
+</instances>
+<busses>
+</busses>
+<nets>
+<net name="GND" class="0">
+<segment>
+<pinref part="X5" gate="G$1" pin="GND"/>
+<wire x1="76.2" y1="93.98" x2="71.12" y2="93.98" width="0.1524" layer="91"/>
+<wire x1="71.12" y1="93.98" x2="71.12" y2="91.44" width="0.1524" layer="91"/>
+<pinref part="GND32" gate="1" pin="GND"/>
+</segment>
+</net>

Commit message: Updated schematic
Connections:
- removed net BB_AIN1: C2.1, R4.1, R5.2
- removed net BB_AIN2: C9.1, R26.1, R27.2
- removed net N$14: R7.1
- removed net N$15: R6.1
- removed net N$34: R31.1
- removed net N$37: R32.1
- new net BB_AIN_E: C9.1, R26.1, R27.2, X1.AIN3
- new net BB_AIN_H: C2.1, R4.1, R5.2, X1.AIN5
- new net BB_DOUT_DOWN: R31.1, X1.GPIO0_27
- new net BB_DOUT_LEFT: R6.1, X1.GPIO1_13
- new net BB_DOUT_RIGHT: R7.1, X1.EHRPWM2B
- new net BB_DOUT_UP: R32.1, X1.GPIO1_15
- new net N$41: X1.EHRPWM2A
- new net N$42: X1.GPIO1_14
- new net N$43: X1.GPIO0_26
- new net N$44: X1.GPIO1_12
Other:
- note added: "BeagleBone headers"
- note added: "P8.11"
- note added: "P8.12"
- note added: "P8.13"
- note added: "P8.14"
- note added: "P8.15"
- note added: "P8.16"
- note added: "P8.17"
- note added: "P8.18"
- note added: "P8.19"
- note added: "P9.36"
- note added: "P9.38"
- note removed: "BeagleBone Headers"
Changed lines of the file:
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@@
 <drawing>
 <settings>
-<setting alwaysvectorfont="no"/>
+<setting alwaysvectorfont="yes"/>
 <setting verticaltext="up"/>
 </settings>
@@
 <sheet>
 <plain>
-<text x="179.07" y="20.32" size="2.54" layer="94">BeagleBone Headers</text>
-<text x="147.32" y="147.32" size="1.778" layer="97">- Power supply is provided by BeagleBone Black</text>
-<text x="147.32" y="152.4" size="2.54" layer="97">Information:</text>
-<text x="147.32" y="142.24" size="1.778" layer="97">- BeagleBone Black cape layout is provided by Adafruit</text>
+<text x="179.07" y="20.32" size="2.54" layer="94">BeagleBone headers</text>
+<text x="162.56" y="93.98" size="1.778" layer="97">- Power supply is provided by BeagleBone Black</text>
+<text x="162.56" y="99.06" size="2.54" layer="97">Information:</text>
+<text x="162.56" y="88.9" size="1.778" layer="97">- BeagleBone Black cape layout is provided by Adafruit</text>
 <text x="10.16" y="63.5" size="1.778" layer="97">P9.17</text>
 <text x="149.86" y="63.5" size="1.778" layer="97">P9.18</text>
@@
 <text x="10.16" y="45.72" size="1.778" layer="97">P9.31</text>
 <text x="149.86" y="50.8" size="1.778" layer="97">P9.28</text>
+<text x="17.78" y="137.16" size="1.778" layer="97">P8.11</text>
+<text x="17.78" y="134.62" size="1.778" layer="97">P8.13</text>
+<text x="17.78" y="132.08" size="1.778" layer="97">P8.15</text>
+<text x="17.78" y="129.54" size="1.778" layer="97">P8.17</text>
+<text x="17.78" y="127" size="1.778" layer="97">P8.19</text>
+<text x="152.4" y="137.16" size="1.778" layer="97">P8.12</text>
+<text x="152.4" y="134.62" size="1.778" layer="97">P8.14</text>
+<text x="152.4" y="132.08" size="1.778" layer="97">P8.16</text>
+<text x="152.4" y="129.54" size="1.778" layer="97">P8.18</text>
+<text x="149.86" y="40.64" size="1.778" layer="97">P9.36</text>
+<text x="149.86" y="38.1" size="1.778" layer="97">P9.38</text>
 </plain>
 <instances>
@@
 <wire x1="53.34" y1="48.26" x2="22.86" y2="48.26" width="0.1524" layer="91"/>
 <label x="22.86" y="48.26" size="1.778" layer="95"/>
+</segment>
+</net>
+<net name="BB_DOUT_RIGHT" class="0">
+<segment>
+<pinref part="X1" gate="G$1" pin="EHRPWM2B"/>
+<wire x1="53.34" y1="134.62" x2="25.4" y2="134.62" width="0.1524" layer="91"/>
+<label x="25.4" y="134.62" size="1.778" layer="95"/>
+</segment>
+</net>
+<net name="BB_DOUT_DOWN" class="0">
+<segment>
+<pinref part="X1" gate="G$1" pin="GPIO0_27"/>
+<wire x1="25.4" y1="129.54" x2="53.34" y2="129.54" width="0.1524" layer="91"/>
+<label x="25.4" y="129.54" size="1.778" layer="95"/>
+</segment>
+</net>
+<net name="N$41" class="0">
+<segment>
+<pinref part="X1" gate="G$1" pin="EHRPWM2A"/>
+<wire x1="53.34" y1="127" x2="25.4" y2="127" width="0.1524" layer="91"/>
+<label x="25.4" y="127" size="1.778" layer="95"/>
+</segment>
+</net>
+<net name="N$42" class="0">
+<segment>
+<pinref part="X1" gate="G$1" pin="GPIO1_14"/>
+<wire x1="109.22" y1="132.08" x2="149.86" y2="132.08" width="0.1524" layer="91"/>
+<label x="124.46" y="132.08" size="1.778" layer="95"/>
+</segment>
+</net>
+<net name="N$43" class="0">
+<segment>
+<pinref part="X1" gate="G$1" pin="GPIO0_26"/>
+<wire x1="149.86" y1="134.62" x2="109.22" y2="134.62" width="0.1524" layer="91"/>
+<label x="124.46" y="134.62" size="1.778" layer="95"/>
+</segment>
+</net>
+<net name="N$44" class="0">
+<segment>
+<pinref part="X1" gate="G$1" pin="GPIO1_12"/>
+<wire x1="109.22" y1="137.16" x2="149.86" y2="137.16" width="0.1524" layer="91"/>
+<label x="124.46" y="137.16" size="1.778" layer="95"/>
+</segment>
+</net>
+<net name="BB_DOUT_LEFT" class="0">
+<segment>
+<pinref part="X1" gate="G$1" pin="GPIO1_13"/>
+<wire x1="25.4" y1="137.16" x2="53.34" y2="137.16" width="0.1524" layer="91"/>
+<label x="25.4" y="137.16" size="1.778" layer="95"/>
+</segment>
+</net>
+<net name="BB_DOUT_UP" class="0">
+<segment>
+<pinref part="X1" gate="G$1" pin="GPIO1_15"/>
+<wire x1="53.34" y1="132.08" x2="25.4" y2="132.08" width="0.1524" layer="91"/>
+<label x="25.4" y="132.08" size="1.778" layer="95"/>
+</segment>
+</net>
+<net name="BB_AIN_H" class="0">
+<segment>
+<pinref part="X1" gate="G$1" pin="AIN5"/>
+<wire x1="109.22" y1="40.64" x2="142.24" y2="40.64" width="0.1524" layer="91"/>
+<label x="119.38" y="40.64" size="1.778" layer="95"/>
+</segment>
+</net>
+<net name="BB_AIN_E" class="0">
+<segment>
+<pinref part="X1" gate="G$1" pin="AIN3"/>
+<wire x1="142.24" y1="38.1" x2="109.22" y2="38.1" width="0.1524" layer="91"/>
+<label x="119.38" y="38.1" size="1.778" layer="95"/>
 </segment>
 </net>
@@
 </segment>
 </net>
-<net name="BB_AIN1" class="0">
+<net name="BB_AIN_H" class="0">
 <segment>
 <pinref part="C2" gate="G$1" pin="1"/>
@@
 </segment>
 </net>
-<net name="N$14" class="0">
+<net name="BB_DOUT_RIGHT" class="0">
 <segment>
 <wire x1="172.72" y1="96.52" x2="144.78" y2="96.52" width="0.1524" layer="91"/>
@@
 </segment>
 </net>
-<net name="N$15" class="0">
+<net name="BB_DOUT_LEFT" class="0">
 <segment>
 <wire x1="170.18" y1="147.32" x2="144.78" y2="147.32" width="0.1524" layer="91"/>
@@
 </segment>
 </net>
-<net name="BB_AIN2" class="0">
+<net name="BB_AIN_E" class="0">
 <segment>
 <pinref part="R26" gate="G$1" pin="1"/>
@@
 </segment>
 </net>
-<net name="N$34" class="0">
+<net name="BB_DOUT_DOWN" class="0">
 <segment>
 <pinref part="R31" gate="G$1" pin="1"/>
@@
 </segment>
 </net>
-<net name="N$37" class="0">
+<net name="BB_DOUT_UP" class="0">
 <segment>
 <pinref part="R32" gate="G$1" pin="1"/>

Commit message: Updated eagle schematic
Parts:
- removed X4: DSUB9, con-te-dsub:DSUB9
- added Q5: SQ2348ES-T1-GE3, vishay_sq2348eS-t1-ge3:SQ2348ES-T1-GE3
- added R33: 1M, rcl:R-EU_R0805
- added R34: 100, rcl:R-EU_R0805
Connections:
- new net N$14: Q5.D, X5.GND
- new net N$23: Q5.G, R33.2, R34.2
- new net N$24: R34.1
- net +5V: now also X5.VCC
- net GND: now also Q5.S, R33.1; no longer X3.6, X3.7, X3.8, X3.9, X4.6, X4.7, X4.8, X4.9, X5.GND
- net N$2: now also IC1D.+IN; no longer IC1A.+IN
- net N$3: now also IC1D.OUT; no longer IC1A.OUT
- net N$5: now also IC1D.-IN; no longer IC1A.-IN
- net ROT_E_DOWN: no longer X4.2
- net ROT_E_POSITION: now also X3.1; no longer X4.5
- net ROT_E_SPEED: no longer X4.4
- net ROT_E_UP: no longer X4.1
- net ROT_H_LEFT: now also X3.3; no longer X3.1
Other:
- note added: "(Coil needs 100 mA continuous)"
- note added: "USB connector for AC power supply switch"
- note removed: "USB-Buchse für Master-Slave Steckdosenleiste"
- moved on the sheet: X3, X5

Commit message: Added DCDC to eagle schematic and made first draft of layout
Parts:
- removed C4, C5, C6, C8: 100n, rcl:C-EUC0603
- removed IC3: MAX3232ESE, maxim:MAX3232ESE
- removed IC4: TLC2264CDU, ti-tlc2264cd:TLC2264CDU
- removed IC5: MCP4901, microchip_mcp4901:MCP4901
- removed R1, R14, R22, R23, R24, R25, R8: 100, rcl:R-EU_R0805
- removed R15: 0, rcl:R-EU_R0805
- removed R16: 5k, rcl:R-EU_R0805
- removed R17: 10k, rcl:R-EU_R0805
- removed X2, X3: DSUB9, con-te-dsub:DSUB9
- added Q6: SQ2348ES-T1-GE3, vishay_sq2348eS-t1-ge3:SQ2348ES-T1-GE3
- added R35: 1M, rcl:R-EU_R0805
- added R36: 100, rcl:R-EU_R0805
- added R37, R38, R39, R40: 10k, rcl:R-EU_R0805
- added U1: TMH0512S, traco_dcdc:TMH0512S
- added X4: DSUB9, con-te-dsub:DSUB9
Connections:
- removed net BB_UART4_RX: R1.1, X1.UART4_RXD
- removed net BB_UART4_TX: R8.1, X1.UART4_TXD
- removed net N$16: C1.1, IC3G$1.C2+
- removed net N$17: C1.2, IC3G$1.C2-
- removed net N$18: C3.2, IC3G$1.C1-
- removed net N$19: C3.1, IC3G$1.C1+
- removed net N$20: C4.1, IC3G$1.V-
- removed net N$21: C5.1, IC3G$1.V+
- removed net N$22: IC3G$1.T1IN, R8.2
- removed net N$24: R34.1
- removed net N$25: IC3G$1.R1OUT, R1.2
- removed net N$27: IC5.SDI, R23.2
- removed net N$28: IC5.SCK, R24.2
- removed net N$29: IC5.!CS, R25.2
- removed net N$30: R22.1
- removed net N$31: IC4A.+IN, IC5.VOUT
- removed net N$32: IC4A.OUT, R14.1, R16.2
- removed net N$33: IC4A.-IN, R16.1, R17.2
- removed net N$4: IC5.!LDAC, R15.2, R22.2
- removed net ROT_E_SPEED: R14.2
- removed net RS232_RX: IC3G$1.R1IN
- removed net RS232_TX: IC3G$1.T1OUT
- new net +12V: R39.2, R40.2, U1.OUT+
- new net ELEVATION_ROTOR_INTERFACE_SUPPLY: R36.1, X1.GPIO2_6
- new net N$34: Q6.G, R35.2, R36.2
- new net N$37: Q6.D, U1.IN-
- new net ROTOR_AC_SUPPLY: R34.1, X1.GPIO1_6
- net +3V3: no longer C6.1, C8.1, IC3P.VCC, IC5.VDD, IC5.VREF
- net +5V: now also C1.1, C3.1, IC6P.V+, R37.2, R38.2, U1.IN+; no longer IC4P.V+
- net BB_SPI1_CS0: no longer R25.1
- net BB_SPI1_D0: no longer R23.1
- net BB_SPI1_SCLK: no longer R24.1
- net GND: now also C1.2, C3.2, IC6P.V-, Q6.S, R35.1, U1.OUT-, X4.6; no longer C4.2, C5.2, C6.2, C8.2, IC3P.GND, IC4P.V-, IC5.VSS, R15.1, R17.1
- net ROT_E_DOWN: now also R37.1, R40.1
- net ROT_E_POSITION: now also X4.1; no longer X3.1
- net ROT_E_UP: now also R38.1, R39.1
- net ROT_H_LEFT: now also X4.3; no longer X3.3
- net ROT_H_POSITON: now also X4.5; no longer X3.5
- net ROT_H_RIGHT: now also X4.2; no longer X3.2
- net ROT_H_SPEED: now also X4.4; no longer X3.4
Other:
- note added: "Elevation rotor interface supply"
- note added: "P9.42"
- note added: "Rotor AC power supply control"
- note added: "Rotor connectors"
- note added: "There is a relay built into the Create ERC-5A which toggles control between this board and the manual switches. It is powerd by this 12V supply. - DC/DC on > Interface control - DC/DC off > Manual control"
- note removed: "Information: - the serial port is deactivated in normal operation"
- note removed: "RS-232 interface"
- note removed: "Rotor controller supply control"
